File: kicad/ilomusiali.kicad_pcb (KiCad board)
At the start: 2 copper layers, 64 x 84.5 mm, 83 parts, among them J1 FPC/0.5mm/bottom contact, J2 2.54mmTP, J3 A01SB141B1, J4 SHOU_HAN_TF_PUSH, J5 2xAA/ZH1.5, Q1 AO3400A, Q3 AO3400A, Q4 AO3401A, SW1 6x3.5x4.3, SW10 6x3.5x4.3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

Commit message: electronics: Completed layout for PCB rev0
Parts:
- added G***: LOGO, project_components:sadale, B.Cu at (156.6, 54.8)
- added NT1: NetTie_2, project_components:NetTie-2_SMD_Pad0.2mm, F.Cu at (151.2, 72.5)
- U1: footprint Package_DFN_QFN:QFN-20-1EP_3x3mm_P0.4mm_EP1.65x1.65mm_ThermalVias -> Package_DFN_QFN:QFN-20-1EP_3x3mm_P0.4mm_EP1.65x1.65mm
- moved D5 12.3 mm to (137.9, 94.1), turned to 0 degrees
- moved D1 11.9 mm to (137.4, 82.6), turned to 0 degrees
- moved D9 11.6 mm to (135.8, 103.0), turned to 0 degrees
- moved R3 4.69 mm to (155.0, 77.9), turned to 180 degrees
- moved C1 3.98 mm to (157.2, 73.9)
- moved C2 3.50 mm to (157.2, 72.4), turned to 0 degrees
- moved R4 2.10 mm to (179.6, 85.2)
- moved D20 2.10 mm to (179.4, 83.5)
- moved J3 2.00 mm to (121.0, 59.0)
- moved R1 2.00 mm to (158.0, 77.9)
- moved SW18 2.00 mm to (120.2, 90.4)
- moved Q1 1.60 mm to (156.2, 80.4)
- moved D19 1.35 mm to (126.6, 89.8), turned to 90 degrees
- moved J4 1.10 mm to (126.3, 75.5)
- moved SW17 1.08 mm to (139.7, 75.0)
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Connections:
- C1 pad 1: GND -> GND2
- C2 pad 2: GND -> GND2
- Y1 pad 2: GND -> GND2
- Y1 pad 4: GND -> GND2
Routing:
- net +5V: track 0.00 -> 157.9 mm, vias 0 -> 1
- net +3V3: track 0.00 -> 134.4 mm, vias 0 -> 6
- net BTN2: track 0.00 -> 122.0 mm
- net BTN1: track 0.00 -> 117.0 mm, vias 0 -> 4
- net BTN0: track 0.00 -> 109.5 mm, vias 0 -> 2
- net BTN3: track 0.00 -> 96.3 mm
- net BTN4: track 0.00 -> 84.1 mm, vias 0 -> 2
- net SPI_MOSI: track 0.00 -> 66.9 mm, vias 0 -> 2
- net SPI_SCK: track 0.00 -> 60.3 mm
- net GND: track 0.00 -> 59.8 mm, vias 0 -> 18
- net BUZZER: track 0.00 -> 57.2 mm
- net SWIO: track 0.00 -> 53.8 mm, vias 0 -> 2
- net GND2: track 0.00 -> 50.6 mm, vias 0 -> 18
- net LCD_CS: track 0.00 -> 44.6 mm, vias 0 -> 4
- net MCU_NRST: track 0.00 -> 41.0 mm
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- added copper zone on B.Cu, net GND
- added copper zone on B.Cu, net GND2
Other:
- outline, holes or cut-outs redrawn
- board text added: "+"
- board text added: "5V"
- board text added: "BAT"
- board text added: "GND"
- board text added: "NRST"
- board text added: "PCB rev0"
- board text added: "SWIO"
- board text added: "USB"
- board text added: "ilo musi 8"
- board text added: "ilo ni li pali pi jan Sate"
- board text added: "ilomusi8.sadale.net"
- board text added: "lupa kalama"
- board text added: "wawa linja"
- board text added: "wawa poki"
