File: kicad/ilomusiali.kicad_pcb (KiCad board)
At the start: 2 copper layers, 64 x 84.5 mm, 85 parts, among them J1 FPC/0.5mm/bottom contact, J2 2.54mmTP, J3 A01SB141B1, J4 SHOU_HAN_TF_PUSH, J5 2xAA/ZH1.5, Q1 AO3400A, Q3 AO3400A, Q4 AO3401A, SW1 6x3.5x4.3, SW10 6x3.5x4.3, SW11 6x3.5x4.3, SW12 6x3.5x4.3, SW13 6x3.5x4.3, SW14 6x3.5x4.3, SW15 6x3.5x4.3, SW16 6x3.5x4.3, SW17 6x3.5x4.3, SW18 SK12D07VG4, SW2 6x3.5x4.3, SW3 6x3.5x4.3, SW4 6x3.5x4.3, SW5 6x3.5x4.3, SW6 6x3.5x4.3, SW7 6x3.5x4.3, SW8 6x3.5x4.3, SW9 6x3.5x4.3, U1 CH32V006F8U6, U3 TX4310B, Y1 24M/CL=12pf

Commit message: electronics: PCB rev1: Using KiCAD 10; Added silkmark for indicating the buzzer position and polarity of the battery connector; With KiCAD 10, the default SOD-323 footprint pads have been shrunken
Parts:
- D19, D20: footprint project_components:D_SOD-323_LargePads -> Diode_SMD:D_SOD-323
Other:
- board text added: "- +"
- board text added: "G"
- board text added: "PCB rev1"
- board text added: "S"
- board text added: "not polarized"
- board text removed: "PCB rev0"

Commit message: electronics: PCB rev1: Added schematics PDF. Changed MCU from CH32V006F8U6 to CH32V006F8U7
Parts:
- U1: value CH32V006F8U6 -> CH32V006F8U7
Changed lines of the file:
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@@
 			)
 		)
-		(property "Value" "CH32V006F8U6"
+		(property "Value" "CH32V006F8U7"
 			(at 0 2.83 180)
 			(layer "F.Fab")
@@
 			)
 		)
-		(property "Datasheet" "https://www.wch-ic.com/products/CH32V003.html"
+		(property "Datasheet" "https://www.wch-ic.com/products/CH32V006.html"
 			(at 0 0 180)
 			(layer "F.Fab")
@@
 			)
 		)
-		(property "Description" "CH32V003 series are industrial-grade general-purpose microcontrollers designed based on 32-bit RISC-V instruction set and architecture. It adopts QingKe V2A core, RV32EC instruction set, and supports 2 levels of interrupt nesting. The series are mounted with rich peripheral interfaces and function modules. Its internal organizational structure meets the low-cost and low-power embedded application scenarios."
+		(property "Description" "CH32V006 series are industrial-grade general-purpose microcontrollers designed based on 32-bit RISC-V instruction set and architecture. It adopts QingKe V2A core, RV32EC instruction set, and supports 2 levels of interrupt nesting. The series are mounted with rich peripheral interfaces and function modules. Its internal organizational structure meets the low-cost and low-power embedded application scenarios."
 			(at 0 0 180)
 			(layer "F.Fab")
@@
 			)
 		)
-		(property "LCSC" "C42431288"
+		(property "LCSC" "C55112440"
 			(at 0 0 180)
 			(unlocked yes)
