File: kicad/ilomusiali.kicad_sch (KiCad schematic)
At the start: 84 parts, among them J1 FPC/0.5mm/bottom contact, J2 2.54mmTP, J3 A01SB141B1, J4 SHOU_HAN_TF_PUSH, J5 2xAA/ZH1.5, Q1 AO3400A, Q3 AO3400A, Q4 AO3401A, SW1 6x3.5x4.3, SW10 6x3.5x4.3, SW11 6x3.5x4.3, SW12 6x3.5x4.3, SW13 6x3.5x4.3, SW14 6x3.5x4.3, SW15 6x3.5x4.3, SW16 6x3.5x4.3, SW17 6x3.5x4.3, SW18 SK12D07VG4, SW2 6x3.5x4.3, SW3 6x3.5x4.3, SW4 6x3.5x4.3, SW5 6x3.5x4.3, SW6 6x3.5x4.3, SW7 6x3.5x4.3, SW8 6x3.5x4.3, SW9 6x3.5x4.3, U1 CH32V006F8U6, U3 TX4310B, Y1 24M/CL=12pf

Commit message: electronics: PCB rev1: Using KiCAD 10; Added silkmark for indicating the buzzer position and polarity of the battery connector; With KiCAD 10, the default SOD-323 footprint pads have been shrunken
Parts:
- D19, D20: footprint project_components:D_SOD-323_LargePads -> Diode_SMD:D_SOD-323
- J3: FT Position Offset 0.0,-0.254 -> 0.0,-0.508; FT Rotation Offset (none) -> -90
Connections:
- net GND: now also J3.SH (Shield), J4.SH (SHIELD); no longer J3.6 (Shield), J4.10 (SHIELD)

Commit message: electronics: PCB rev1: Added schematics PDF. Changed MCU from CH32V006F8U6 to CH32V006F8U7
Parts:
- U1: value CH32V006F8U6 -> CH32V006F8U7; LCSC C42431288 -> C55112440
Changed lines of the file:
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@@
 	(title_block
 		(title "ilo musi 8")
-		(rev "0")
+		(rev "1")
 	)
 	(rectangle
@@
 			)
 		)
-		(property "Value" "CH32V006F8U6"
+		(property "Value" "CH32V006F8U7"
 			(at 59.2933 62.23 0)
 			(show_name no)
@@
 			)
 		)
-		(property "Datasheet" "https://www.wch-ic.com/products/CH32V003.html"
+		(property "Datasheet" "https://www.wch-ic.com/products/CH32V006.html"
 			(at 55.88 80.01 0)
 			(hide yes)
@@
 			)
 		)
-		(property "Description" "CH32V003 series are industrial-grade general-purpose microcontrollers designed based on 32-bit RISC-V instruction set and architecture. It adopts QingKe V2A core, RV32EC instruction set, and supports 2 levels of interrupt nesting. The series are mounted with rich peripheral interfaces and function modules. Its internal organizational structure meets the low-cost and low-power embedded application scenarios."
+		(property "Description" "CH32V006 series are industrial-grade general-purpose microcontrollers designed based on 32-bit RISC-V instruction set and architecture. It adopts QingKe V2A core, RV32EC instruction set, and supports 2 levels of interrupt nesting. The series are mounted with rich peripheral interfaces and function modules. Its internal organizational structure meets the low-cost and low-power embedded application scenarios."
 			(at 57.15 80.01 0)
 			(hide yes)
@@
 			)
 		)
-		(property "LCSC" "C42431288"
+		(property "LCSC" "C55112440"
 			(at 57.15 80.01 0)
 			(hide yes)
